File: kicad/my_rp60.kicad_pcb (KiCad board)
At the start: 2 copper layers, 285 x 95.8 mm, 156 parts, among them SW1 SW_Push, SW2 SW_Push, U3 RP2040, U4 TLV73333PDBV, U5 W25Q128JVS, Y1 Crystal_GND24

Commit message: kicad: oneside pcb
Parts:
- removed SW1, SW2: SW_Push, Button_Switch_SMD:SW_SPST_Omron_B3FS-100xP
- added ?: , , F.Cu at (237.8, 126.2)
- added ?: , , F.Cu at (242.5, 132.5)
- added ?: , , F.Cu at (221.5, 132.5)
- added ?: , , F.Cu at (241.5, 126.2)
- added ?: , , F.Cu at (226.0, 132.5)
- added ?: , , F.Cu at (238.0, 132.5)
- added ?: , , F.Cu at (186.8, 134.7)
- added ?: , , F.Cu at (221.5, 126.0)
- added ?: , , F.Cu at (226.0, 126.0)
- C1, C10, C13, C15, C16, C17, C18, C19, C2, C3, C4, C5, C6, C7, C8, C9, R3, R4, R5, R6, R7, U3, U4, U5, Y1: moved to B.Cu
- moved C5 18.1 mm to (207.6, 139.8), turned to 0 degrees
- moved R6 17.5 mm to (221.4, 123.8)
- moved R5 15.6 mm to (198.2, 123.1)
- moved C17 15.5 mm to (192.4, 123.2)
- moved C8 13.7 mm to (202.6, 137.8), turned to -90 degrees
- moved C9 13.7 mm to (201.5, 137.8), turned to -90 degrees
- moved C15 12.0 mm to (192.5, 136.9), turned to 90 degrees
- moved C16 12.0 mm to (197.3, 136.9), turned to 90 degrees
- moved C10 11.3 mm to (199.9, 136.6)
- moved U4 11.0 mm to (194.9, 136.4)
- moved C13 9.21 mm to (199.4, 135.5)
- moved U5 8.51 mm to (196.5, 126.7)
- moved C4 7.51 mm to (202.7, 127.2), turned to 90 degrees
- moved C6 7.31 mm to (207.0, 127.0), turned to 90 degrees
- moved R4 7.08 mm to (199.4, 134.5)
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Connections:
- D_- pad 1: r4 -> (no net)
- D_[ pad 1: r4 -> (no net)
- REF** pad 1: GND -> (no net)
- U3 pad 11: r4 -> (no net)
- U3 pad 12: c12 -> r2
- U3 pad 13: c11 -> c8
- U3 pad 14: c10 -> c9
- U3 pad 27: c9 -> (no net)
- U3 pad 28: c8 -> (no net)
- U3 pad 29: r2 -> (no net)
- U3 pad 3: MOTION -> c6
- U3 pad 30: r1 -> c10
- U3 pad 31: r3 -> c11
- U3 pad 32: c7 -> c12
- U3 pad 34: r0 -> r4
- U3 pad 35: c6 -> c5
- U3 pad 36: c0 -> c4
- U3 pad 37: c1 -> (no net)
- U3 pad 38: c2 -> c3
- U3 pad 39: c3 -> c2
- U3 pad 4: SCLK -> r0
- U3 pad 40: c4 -> c1
- U3 pad 41: c5 -> c0
- U3 pad 5: MOSI -> c7
- U3 pad 6: MISO -> (no net)
- U3 pad 7: Net-(U3-Pad7) -> (no net)
- U3 pad 8: Net-(U3-Pad8) -> r3
- U3 pad 9: Net-(U3-Pad9) -> r1
- USB pad A6: (no net) -> D+
- USB pad A7: (no net) -> D-
Routing:
- net Net-(R6-Pad2): track 27.1 -> 11.5 mm
- net c5: track 126.9 -> 141.0 mm, vias 1 -> 2
- net c3: track 166.4 -> 179.1 mm, vias 1 -> 2
- net c4: track 143.6 -> 154.6 mm, vias 1 -> 3
- net c2: track 206.9 -> 217.8 mm, vias 1 -> 2
- net QSPI_SS: track 40.5 -> 29.7 mm
- net c1: track 235.9 -> 245.6 mm, vias 1 -> 2
- net c0: track 250.2 -> 259.2 mm, vias 1 -> 2
- net +5V: track 277.6 -> 270.3 mm
- net r2: track 384.4 -> 390.5 mm, vias 1 -> 2
- net r1: track 411.7 -> 416.3 mm, vias 1 -> 2
- net c8: track 155.8 -> 159.1 mm, vias 0 -> 1
- net r3: track 360.4 -> 363.7 mm
- net c7: track 86.4 -> 89.0 mm, vias 0 -> 1
- net r0: track 424.7 -> 427.2 mm, vias 1 -> 2
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- added copper zone on B.Cu, net +1V1
- added copper zone on B.Cu, net +3V3
- removed copper zone on F.Cu, net +1V1
- removed copper zone on F.Cu, net +3V3
Other:
- board text added: "C00 = 41 C07 = 05 C01 = 40 C08 = 13 C02 = 39 C09 = 14 C03 = 38 C10 = 30 C04 = 36 XXXXXXXX C05 = 35 C11 = 31 C06 = 03 C12 = 32"
- board text added: "R00 = 04 R01 = 09 R02 = 12 R03 = 08 R04 = 34"
- board text removed: "C00 = 36 C07 = 32 C01 = 37 C08 = 28 C02 = 38 C09 = 27 C03 = 39 C10 = 14 C04 = 40 XXXXXXXX C05 = 41 C11 = 13 C06 = 35 C12 = 12"
- board text removed: "R00 = 34 R01 = 30 R02 = 29 R03 = 31 R04 = 11"
